File: Hardware/MOPS-Hub_Readout_board/FTDI.kicad_sch (KiCad schematic)
At the start: 50 parts, among them U1 TPS73633DBV, U2 93LCxxB, U3 FT2232HL, Y1 12MHz

Commit message: Flash footprint changed to TSSOP-8
Parts:
- U2: footprint Package_SO:SOIC-8_3.9x4.9mm_P1.27mm -> Package_SO:TSSOP-8_4.4x3mm_P0.65mm
Changed lines of the file:
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@@
 			)
 		)
-		(property "Footprint" "Package_SO:SOIC-8_3.9x4.9mm_P1.27mm"
+		(property "Footprint" "Package_SO:TSSOP-8_4.4x3mm_P0.65mm"
 			(at 96.52 114.3 0)
 			(effects
